File: projects/cvra_actuator_board/version_current/working/working.kicad_pcb (KiCad board)
At the start: 4 copper layers, 22 x 40 mm, 62 parts, among them J1 SERVO DCDC 5V, J10 Servo, J2 Conn_01x06, J3 Actuator1, J4 Actuator2, J5 SWD/DEBUG, J6 BATTERY, J7 CAN, J8 CAN, J9 Servo, U1 STM32F302K8U6, U2 MCP1703, U3 MAX3051, U4 MPRLS0015PA0000SA, U5 MPRLS0015PA0000SA, U6 DRV8847_TSSOP, X1 16MHz 10ppm

Commit message: updated all projects from src
Other:
- net class Default added: clearance 0.1524, trace_width 0.1524, via_dia 0.5, via_drill 0.2

Commit message: some generations
Other:
- net class Default removed
