File: projects/electroniccats_meditemp/version_current/working/working.kicad_pcb (KiCad board)
At the start: 2 copper layers, 100 x 100 mm, 56 parts, among them J1 HC-SR04, J10 Screw_Terminal_01x03, J11 Screw_Terminal_01x03, J2 FTDI, J3 LCD, J4 MLX90614, J5 DS1307, J6 SD, J7 Screw_Terminal_01x02, J8 Screw_Terminal_01x11, J9 Screw_Terminal_01x11, Q1 MMBT2222A, Q2 MMBT2222A, Q3 MMBT2222A, SW1 RST, SW2 BOOT, SW3 Extra, U1 AZ1084CD-5.0TRG1, U2 AP2114H-3.3TRG1, U3 ESP32-WROOM-32, U4 LTV-817, U5 LTV-817, Y1 UD2-3NU, Y2 UD2-3NU

Commit message: updated all projects from src
Other:
- net class Default added: clearance 0.2, trace_width 0.3, via_dia 0.8, via_drill 0.4
- net class V+ added: clearance 0.2, trace_width 0.5, via_dia 0.8, via_drill 0.4

Commit message: converted omerk brd to kicad
Other:
- net class Default removed
- net class V+ removed
