File: projects/ai03_2725_jp60/version_current/working/working.kicad_pcb (KiCad board)
At the start: 2 copper layers, 285 x 95.1 mm, 153 parts, among them SW1 SW_Push, U1 ATmega32U4-MU, U2 PRTR5V0U2X, Y1 16MHz

Commit message: updated all projects from src
Other:
- net class Default added: clearance 0.1778, trace_width 0.254, via_dia 0.6, via_drill 0.4
- net class Earth added: clearance 0.1778, trace_width 0.508, via_dia 0.6, via_drill 0.4
- net class Power added: clearance 0.1778, trace_width 0.381, via_dia 0.6, via_drill 0.4
- net class USB added: clearance 0.1778, trace_width 0.261112, via_dia 0.6, via_drill 0.4
