File: projects/ai03_2725_orbit/version_current/working/working.kicad_pcb (KiCad board)
At the start: 2 copper layers, 263.8 x 125 mm, 165 parts, among them J1 PJ-3200B-4A, J11 PJ-3200B-4A, J13 Breakaway_Tabs, J14 Breakaway_Tabs, J17 Breakaway_Tabs, J18 Breakaway_Tabs, J19 Breakaway_Tabs, J3 Breakaway_Tabs, J5 Breakaway_Tabs, J6 Breakaway_Tabs, J7 Breakaway_Tabs, J9 Breakaway_Tabs, SW1 SW_Push, SW2 SW_Push, U1 ATmega32U4-AU, U2 PRTR5V0U2X, U3 ATmega32U4-AU, U4 PRTR5V0U2X, Y1 16MHz, Y2 16MHz

Commit message: updated all projects from src
Other:
- net class Default added: clearance 0.1778, trace_width 0.254, via_dia 0.8, via_drill 0.4
- net class POWER added: clearance 0.1778, trace_width 0.381, via_dia 0.8, via_drill 0.4
