File: projects/ai03_2725_stabilizershims/version_current/working/working.kicad_pcb (KiCad board)
At the start: 2 copper layers, 96 x 83 mm, 96 parts

Commit message: updated all projects from src
Other:
- net class Default added: clearance 0.2, trace_width 0.25, via_dia 0.8, via_drill 0.4
