File: projects/ai03_2725_titan/version_current/working/working.kicad_pcb (KiCad board)
At the start: 2 copper layers, 285.4 x 94.9 mm, 3 parts, among them U1 Outline

Commit message: updated all projects from src
Other:
- net class Default added: clearance 0.2, trace_width 0.25, via_dia 0.6, via_drill 0.4
