File: projects/ai03_2725_voyager60/version_current/working/working.kicad_pcb (KiCad board)
At the start: 2 copper layers, 285 x 95.1 mm, 265 parts, among them Q1 2N7002, SW1 5.2x5.2mm, U1 ATmega32U4-MU, U2 PRTR5V0U2X, Y1 16Mhz

Commit message: updated all projects from src
Other:
- net class Default added: clearance 0.2032, trace_width 0.254, via_dia 0.6, via_drill 0.4
- net class Power added: clearance 0.2032, trace_width 0.381, via_dia 0.6, via_drill 0.4
