File: projects/alasofia_model_v/version_current/working/working.kicad_pcb (KiCad board)
At the start: 2 copper layers, 242.9 x 76.2 mm, 122 parts, among them SW1 SW_Push, U1 ATmega32U4-MU, U2 PRTR5V0U2X, Y1 16MHz

Commit message: updated all projects from src
Other:
- net class Default added: clearance 0.2, trace_width 0.25, via_dia 0.8, via_drill 0.4
