File: projects/asukiaaa_i2cbrushlessmotors/version_current/working/working.kicad_pcb (KiCad board)
At the start: 2 copper layers, 50 x 50 mm, 65 parts, among them J1 Conn_01x03, J2 Conn_01x06, J3 Header, J4 Socket, J5 Conn_01x03, Q1 Q_PMOS_GSD, Q10 Q_PMOS_GSD, Q11 Q_NMOS_GSD, Q12 Q_NMOS_GSD, Q13 Q_PMOS_GSD, Q14 Q_NMOS_GSD, Q15 Q_NMOS_GSD, Q16 Q_PMOS_GSD, Q17 Q_NMOS_GSD, Q18 Q_NMOS_GSD, Q2 Q_NMOS_GSD, Q3 Q_NMOS_GSD, Q4 Q_PMOS_GSD, Q5 Q_NMOS_GSD, Q6 Q_NMOS_GSD, Q7 Q_PMOS_GSD, Q8 Q_NMOS_GSD, Q9 Q_NMOS_GSD, U1 ATmega328PB-MU

Commit message: updated all projects from src
Other:
- net class Default added: clearance 0.2, trace_width 0.25, via_dia 0.8, via_drill 0.4
