File: projects/dragonmux_glasgow/version_current/working/working.kicad_pcb (KiCad board)
At the start: 2 copper layers, 207.5 x 45.5 mm, 131 parts, among them J1 AST04106, J10 AST04106, J11 AST04106, J2 DNP, J3 Conn_02x05_Odd_Even, J4 USB_B_Micro, J5 AST04106, J6 Conn_02x05_Odd_Even, J7 AST04106, J8 AST04106, J9 AST04106, Q1 BSS138, Q2 BSS138, U1 TPS3700, U10 TCA9534, U11 74HC4066, U2 74LVC2G14, U3 TPS3700, U4 INA260, U5 TPS3700, U6 74LVC2G14, U7 AP2127K-3.3, U8 74HC4066, U9 74HC4066

Commit message: converted omerk brd to kicad
Connections:
- net /port-connection/~Aux_conn_ctrl renamed /port-connection/~{Aux_conn_ctrl}
- net /port-connection/~Port_conn_ctrl renamed /port-connection/~{Port_conn_ctrl}
Other:
- net class Default removed

Commit message: updated all projects from src
Connections:
- net /port-connection/~{Aux_conn_ctrl} renamed /port-connection/~Aux_conn_ctrl
- net /port-connection/~{Port_conn_ctrl} renamed /port-connection/~Port_conn_ctrl
Other:
- net class Default added: clearance 0.2, trace_width 0.2, via_dia 0.7, via_drill 0.3
