File: projects/electrolama_oshcamp23_badge/version_current/working/working.kicad_sch (KiCad schematic)
At the start: 0 parts

Commit message: update
Parts:
- added ANT2: ANT3216LL00R2400A, working:YAGEO-ANT3216LL00R2400A, symbol working-eagle-import:ANT-CERAMIC-YAGEO-ANT3216LL00R2400A
- added C1, C2, C3, C33, C34: 47u, working:_PKG_C_1206, symbol working-eagle-import:CAP-1206
- added C21, C22: TBD, working:_PKG_C_0402_NOTHERMALS, symbol working-eagle-import:CAP-0402-NOTHERMALS
- added C23, C24: 8p, working:_PKG_C_0402, symbol working-eagle-import:CAP-0402
- added C25, C27: 4u7, working:_PKG_C_0402_NOTHERMALS, symbol working-eagle-import:CAP-0402-NOTHERMALS
- added C26, C28, C29, C30, C32: 100n, working:_PKG_C_0402_NOTHERMALS, symbol working-eagle-import:CAP-0402-NOTHERMALS
- added C31, C4, C5, C6: 100n, working:_PKG_C_0402, symbol working-eagle-import:CAP-0402
- added CON1: USBC_USB-C-12, working:USBC_C-31-M-12, symbol working-eagle-import:USBC_USB-C-12
- added CON2: STEMMA_I2C_QT, working:JST_SH4, symbol working-eagle-import:STEMMA_I2C_QT
- added D1: DIODE-SWITCHING-1N4148W, working:_PKG_SOD123, symbol working-eagle-import:DIODE-SWITCHING-1N4148W
- added IC1: INTERFACE-CH343G, working:_PKG_SOP16, symbol working-eagle-import:INTERFACE-CH343G
- added IC2: LD1117-3.3, working:_PKG_SOT223-4_TI-DCY4, symbol working-eagle-import:POWER-LDO-LD1117-SOT223-4
- added IC4: WMCU-ESP8285H16, working:QFN50P500X500X90-33N, symbol working-eagle-import:WMCU-ESP8285H16
- added J1: 6103XX21121_61030621121, working:61030621121, symbol working-eagle-import:6103XX21121_61030621121
- added L2: TBD, working:_PKG_L_0402, symbol working-eagle-import:INDUCTOR-0402
- added LED1: WS2812B5050, working:WS2812B, symbol working-eagle-import:WS2812B5050
- added MOD2: ESP-12S, working:ESP-12S, symbol working-eagle-import:MODULE_ESP-12S
- added P1: Buzzer, working:MLT-8530, symbol working-eagle-import:PIEZO-MLT-8530
- added Q1, Q2, Q3: SS8050, working:SOT96P237X111-3N, symbol working-eagle-import:NPN-MMBT5550LT1G
- added R1: 220, working:_PKG_R_0603, symbol working-eagle-import:RES-0603
- added R12, R13, R14, R15, R16, R17, R4, R5: 12k 1%, working:_PKG_R_0402, symbol working-eagle-import:RES-0402
- added R2, R3: 5k1, working:_PKG_R_0603, symbol working-eagle-import:RES-0603
- added SJ1, SJ2, SJ3, SJ4: SJ-SHORT, working:SJ-SHORT, symbol working-eagle-import:SJ-SHORT
- added SW1, SW2, SW3, SW4, SW5, SW6, SW7: PUSHBUTTON-6X6MM, working:GENERIC_SPNO_4P_6X6MM, symbol working-eagle-import:PUSHBUTTON-6X6MM
- added XT2: 26MHz, working:XTAL-4P-2016, symbol working-eagle-import:XTAL-4P-2016
Connections:
- new net: ANT2.S1 (FEED), C21.2, L2.1
- new net: D1.2 (A), P1.-, Q3.3 (C)
- new net: Q1.1 (B), R5.1
- new net: Q3.1 (B), R1.1
- new net: CON1.CC1, R3.2
- new net: C22.2, IC4.2 (LNA), L2.2
- new net: Q2.1 (B), R4.2
- new net: IC4.31 (RES12K), R12.1
- new net: C5.1, C6.1, IC1.15 (VIO), IC1.4 (V3)
- new net: CON1.CC2, R2.2
- new net AUTORST_BOOT: J1.6, Q1.3 (C), SJ4.1
- new net AUTORST_EN: J1.1, Q2.3 (C), SJ1.2
- new net DTR: IC1.10 (DTR), Q1.2 (E), R4.1
- new net EN: IC4.7 (CHIP_EN), MOD2.EN, R13.2, SJ1.1
- new net GND: C1.2, C2.2, C21.1, C22.1, C23.1, C24.1, C25.1, C26.1, C27.1, C28.1, C29.1, C3.2, C30.1, C31.2, C32.1, C33.2, C34.2, C4.2, C5.2, C6.2, CON1.GND@1 (GND), CON1.GND@2 (GND), CON1.P$1 (CHASSIS), CON1.P$2 (CHASSIS), CON1.P$3 (CHASSIS), CON1.P$4 (CHASSIS), CON1.P$5 (CHASSIS), CON1.P$6 (CHASSIS), CON1.P$7 (CHASSIS), CON1.P$8 (CHASSIS), CON2.1 (GND), IC1.1 (GND), IC2.1 (GND), IC4.33 (GND), J1.4, LED1.3-GND (GND), MOD2.EPAD (GND), MOD2.GND, Q3.2 (E), R12.2, R16.1, R2.1, R3.1, SW1.P$3 (2), SW1.P$4 (2), SW2.P$3 (2), SW2.P$4 (2), SW3.P$3 (2), SW3.P$4 (2), SW4.P$3 (2), SW4.P$4 (2), SW5.P$3 (2), SW5.P$4 (2), SW6.P$3 (2), SW6.P$4 (2), XT2.2, XT2.4
- new net IO0: IC4.15 (GPIO0), MOD2.IO0, R14.2, SJ4.2, SW3.P$1 (1), SW3.P$2 (1)
- new net IO12: CON2.4 (SCL), IC4.10 (MTDI), MOD2.IO12, SW5.P$1 (1), SW5.P$2 (1)
- new net IO13: IC4.12 (MTCK), MOD2.IO13, R1.2
- new net IO14: CON2.3 (SDA), IC4.9 (MTMS), MOD2.IO14, SW6.P$1 (1), SW6.P$2 (1)
- new net IO15: IC4.13 (MTDO), MOD2.IO15, R16.2, SW7.P$1 (1), SW7.P$2 (1)
- new net IO1_TX: IC4.26 (U0TXD), MOD2.TXD/IO1, SJ2.1
- new net IO2: IC4.14 (GPIO2), MOD2.IO2, R15.2, SW4.P$1 (1), SW4.P$2 (1)
- new net IO3_RX: IC4.25 (U0RXD), MOD2.RXD/IO3, SJ3.1
- new net IO4: IC4.16 (GPIO4), MOD2.IO4, SW2.P$1 (1), SW2.P$2 (1)
- new net IO5: IC4.24 (GPIO5), LED1.4-DIN (DI), MOD2.IO5, SW1.P$1 (1), SW1.P$2 (1)
- new net PC_RX: IC1.3 (RXD), J1.3, SJ2.2
- new net PC_TX: IC1.2 (TXD), J1.5, SJ3.2
- new net RST_C: C30.2, IC4.32 (EXT_RSTB), R17.1
- new net RST_M: MOD2.RST
- new net RTS: IC1.11 (RTS), Q2.2 (E), R5.2
- new net USB_N: CON1.DN1, CON1.DN2, IC1.6 (UD-)
- new net USB_P: CON1.DP1, CON1.DP2, IC1.5 (UD+)
- new net VCC: C2.1, C25.2, C26.2, C27.2, C28.2, C29.2, C3.1, C31.1, C32.2, C33.1, C34.1, CON2.2 (V+), D1.1 (C), IC2.2 (VOUT), IC2.4 (TAB), IC4.1 (VDDA_1), IC4.11 (VDDPST_1), IC4.17 (VDDPST_2), IC4.29 (VDDD), IC4.3 (VDD3P3_1), IC4.30 (VDDA_2), IC4.4 (VDD3P3_2), J1.2, LED1.1-VDD (VDD), MOD2.VCC, P1.+, R13.1, R14.1, R15.1, R17.2, SW7.P$3 (2), SW7.P$4 (2)
- new net VUSB: C1.1, C4.1, CON1.VBUS@1 (VBUS), CON1.VBUS@2 (VBUS), IC1.16 (VDD5), IC1.7 (VBUS), IC2.3 (VIN)
- new net XTAL_IN: C23.2, IC4.28 (XTAL_IN), XT2.1
- new net XTAL_OUT: C24.2, IC4.27 (XTAL_OUT), XT2.3
Other:
- removed sheet working_1
- removed sheet working_2
- note added: ""EXT_RSTB serves as the reset pin of ESP8266EX. This pin contains an internal pull-up resistor and is active low." "We recommend that you use CHIP_EN, instead of EXT_RSTB, to reset the chip." -ESP8266 HW Design Guidelines"
- note added: "** Resistors here do not need to be 1% but we are using the 12K 1% that we already have on the BOM to reduce the number of unique items we have on this board."
- note added: "5V -> 3.3V LDO"
- note added: "ANT1"
- note added: "Cut solder jumpers to turn this into an ESP-PROG compatible programmer (isolates the on-board ESP module and chip from CH343 UART)"
- note added: "DTR RTS -> Q1 Q2 EN BOOT 1 1 on on 1 1 0 0 off off 1 1 1 0 on off 0 1 0 1 off on 1 0"
- note added: "ESP Auto-Reset"
- note added: "ESP-12 Module"
- note added: "ESP8285H16 (ESP8266 + SPI FLASH)"
- note added: "I2C Port"
- note added: "IO15 is a bootstrap pin that needs to be pulled high at boot, hence the reason why it is different."
- note added: "Piezo Buzzer"
- note added: "Pushbuttons"
- note added: "RGB LED"
- note added: "This board is designed to be used as part of a solder paste workshop at OSHCamp 2023, also acting as a name badge, a generic sensor device using the qwiic/ stemma qt compatible I2C port and the Tasmota firmware and even a little piece of art, courtesy of OSHUG co-founder Paul Downey. You can also use it as a comically large USB-UART / ESP-Prog adapter for your other designs~ You'll notice both an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"
- note added: "U0RXD"
- note added: "U0TXD"
- note added: "UART/ESP-Prog Header"
- note added: "USB-C + USB-Serial"
- note added: "https://lab.electrolama.com/ob23 This open-source hardware design is licensed under the Solderpad Hardware License 2.0."
