File: projects/electrolama_oshcamp23_badge/version_current/working/working.sch (EAGLE design)
At the start: 58 parts, among them CON2 STEMMA_I2C_QT, IC2 LD1117-3.3, IC4 WMCU-ESP8285H16, J1 61030621121, P1 Buzzer, Q1 SS8050, Q2 SS8050, Q3 SS8050

Commit message: resyncing
Parts:
- removed ANT2: ANT3216LL00R2400A, ok-rf-dev:ANT-CERAMIC-YAGEO-ANT3216LL00R2400A
- removed C21, C22: TBD, ok-discretes-dev:CAP-0402-NOTHERMALS
- removed C23, C24: 8p, ok-discretes-dev:CAP-0402
- removed C25, C27: 4u7, ok-discretes-dev:CAP-0402-NOTHERMALS
- removed C26, C28, C29, C30, C32: 100n, ok-discretes-dev:CAP-0402-NOTHERMALS
- removed C31: 100n, ok-discretes-dev:CAP-0402
- removed C33, C34: 47u, ok-discretes-dev:CAP-1206
- removed IC4: WMCU-ESP8285H16, ok-chips-dev:WMCU-ESP8285H16
- removed L2: TBD, ok-discretes-dev:INDUCTOR-0402
- removed MOD2: ESP-12S, ok-modules-dev:MODULE_ESP-12S
- removed R12, R13, R14, R15, R16, R17: 12k 1%, ok-discretes-dev:RES-0402
- removed XT2: 26MHz, ok-xtal-osc-dev:XTAL-4P-2016
- added ANT1: ANT3216LL00R2400A, ok-rf-dev:ANT-CERAMIC-YAGEO-ANT3216LL00R2400A
- added C10, C18: 47u, ok-discretes-dev:CAP-1206
- added C11, C7: 8p, ok-discretes-dev:CAP-0402
- added C12, C14: 4u7, ok-discretes-dev:CAP-0402-NOTHERMALS
- added C13, C15, C16, C17, C20: 100n, ok-discretes-dev:CAP-0402-NOTHERMALS
- added C19: 100n, ok-discretes-dev:CAP-0402
- added C8, C9: TBD, ok-discretes-dev:CAP-0402-NOTHERMALS
- added IC3: WMCU-ESP8285H16, ok-chips-dev:WMCU-ESP8285H16
- added L1: TBD, ok-discretes-dev:INDUCTOR-0402
- added MOD1: ESP-12S, ok-modules-dev:MODULE_ESP-12S
- added R10, R11, R6, R7, R8, R9: 12k 1%, ok-discretes-dev:RES-0402
- added XT1: 26MHz, ok-xtal-osc-dev:XTAL-4P-2016
Connections:
- removed net ANT'1: ANT2.FEED, C21.2, L2.1
- removed net ANT1: C22.2, IC4.LNA, L2.2
- removed net N$1: IC4.RES12K, R12.1
- new net ANT: C9.2, IC3.LNA, L1.2
- new net ANT': ANT1.FEED, C8.2, L1.1
- new net N$6: IC3.RES12K, R6.1
- net EN: now also IC3.CHIP_EN, MOD1.EN, R7.2; no longer IC4.CHIP_EN, MOD2.EN, R13.2
- net GND: now also C10.2, C11.1, C12.1, C13.1, C14.1, C15.1, C16.1, C17.1, C18.2, C19.2, C20.1, C7.1, C8.1, C9.1, IC3.GND, MOD1.GND, R10.1, R6.2, XT1.2, XT1.4; no longer C21.1, C22.1, C23.1, C24.1, C25.1, C26.1, C27.1, C28.1, C29.1, C30.1, C31.2, C32.1, C33.2, C34.2, IC4.GND, MOD2.GND, R12.2, R16.1, XT2.2, XT2.4
- net IO0: now also IC3.GPIO0, MOD1.IO0, R8.2; no longer IC4.GPIO0, MOD2.IO0, R14.2
- net IO12: now also IC3.MTDI, MOD1.IO12; no longer IC4.MTDI, MOD2.IO12
- net IO13: now also IC3.MTCK, MOD1.IO13; no longer IC4.MTCK, MOD2.IO13
- net IO14: now also IC3.MTMS, MOD1.IO14; no longer IC4.MTMS, MOD2.IO14
- net IO15: now also IC3.MTDO, MOD1.IO15, R10.2; no longer IC4.MTDO, MOD2.IO15, R16.2
- net IO1_TX: now also IC3.U0TXD, MOD1.TXD/IO1; no longer IC4.U0TXD, MOD2.TXD/IO1
- net IO2: now also IC3.GPIO2, MOD1.IO2, R9.2; no longer IC4.GPIO2, MOD2.IO2, R15.2
- net IO3_RX: now also IC3.U0RXD, MOD1.RXD/IO3; no longer IC4.U0RXD, MOD2.RXD/IO3
- net IO4: now also IC3.GPIO4, MOD1.IO4; no longer IC4.GPIO4, MOD2.IO4
- net IO5: now also IC3.GPIO5, MOD1.IO5; no longer IC4.GPIO5, MOD2.IO5
- net RST_C: now also C20.2, IC3.EXT_RSTB, R11.1; no longer C30.2, IC4.EXT_RSTB, R17.1
- net RST_M: now also MOD1.RST; no longer MOD2.RST
- net VCC: now also C10.1, C12.2, C13.2, C14.2, C15.2, C16.2, C17.2, C18.1, C19.1, IC3.VDD3P3_1, IC3.VDD3P3_2, IC3.VDDA_1, IC3.VDDA_2, IC3.VDDD, IC3.VDDPST_1, IC3.VDDPST_2, MOD1.VCC, R11.2, R7.1, R8.1, R9.1; no longer C25.2, C26.2, C27.2, C28.2, C29.2, C31.1, C32.2, C33.1, C34.1, IC4.VDD3P3_1, IC4.VDD3P3_2, IC4.VDDA_1, IC4.VDDA_2, IC4.VDDD, IC4.VDDPST_1, IC4.VDDPST_2, MOD2.VCC, R13.1, R14.1, R15.1, R17.2
- net XTAL_IN: now also C7.2, IC3.XTAL_IN, XT1.1; no longer C23.2, IC4.XTAL_IN, XT2.1
- net XTAL_OUT: now also C11.2, IC3.XTAL_OUT, XT1.3; no longer C24.2, IC4.XTAL_OUT, XT2.3

Commit message: update
Parts:
- removed ANT1: ANT3216LL00R2400A, ok-rf-dev:ANT-CERAMIC-YAGEO-ANT3216LL00R2400A
- removed C10, C18: 47u, ok-discretes-dev:CAP-1206
- removed C11, C7: 8p, ok-discretes-dev:CAP-0402
- removed C12, C14: 4u7, ok-discretes-dev:CAP-0402-NOTHERMALS
- removed C13, C15, C16, C17, C20: 100n, ok-discretes-dev:CAP-0402-NOTHERMALS
- removed C19: 100n, ok-discretes-dev:CAP-0402
- removed C8, C9: TBD, ok-discretes-dev:CAP-0402-NOTHERMALS
- removed IC3: WMCU-ESP8285H16, ok-chips-dev:WMCU-ESP8285H16
- removed L1: TBD, ok-discretes-dev:INDUCTOR-0402
- removed MOD1: ESP-12S, ok-modules-dev:MODULE_ESP-12S
- removed R10, R11, R6, R7, R8, R9: 12k 1%, ok-discretes-dev:RES-0402
- removed XT1: 26MHz, ok-xtal-osc-dev:XTAL-4P-2016
- added ANT2: ANT3216LL00R2400A, ok-rf-dev:ANT-CERAMIC-YAGEO-ANT3216LL00R2400A
- added C21, C22: TBD, ok-discretes-dev:CAP-0402-NOTHERMALS
- added C23, C24: 8p, ok-discretes-dev:CAP-0402
- added C25, C27: 4u7, ok-discretes-dev:CAP-0402-NOTHERMALS
- added C26, C28, C29, C30, C32: 100n, ok-discretes-dev:CAP-0402-NOTHERMALS
- added C31: 100n, ok-discretes-dev:CAP-0402
- added C33, C34: 47u, ok-discretes-dev:CAP-1206
- added IC4: WMCU-ESP8285H16, ok-chips-dev:WMCU-ESP8285H16
- added L2: TBD, ok-discretes-dev:INDUCTOR-0402
- added MOD2: ESP-12S, ok-modules-dev:MODULE_ESP-12S
- added R12, R13, R14, R15, R16, R17: 12k 1%, ok-discretes-dev:RES-0402
- added XT2: 26MHz, ok-xtal-osc-dev:XTAL-4P-2016
Connections:
- removed net ANT: C9.2, IC3.LNA, L1.2
- removed net ANT': ANT1.FEED, C8.2, L1.1
- removed net N$6: IC3.RES12K, R6.1
- new net ANT'1: ANT2.FEED, C21.2, L2.1
- new net ANT1: C22.2, IC4.LNA, L2.2
- new net N$1: IC4.RES12K, R12.1
- net EN: now also IC4.CHIP_EN, MOD2.EN, R13.2; no longer IC3.CHIP_EN, MOD1.EN, R7.2
- net GND: now also C21.1, C22.1, C23.1, C24.1, C25.1, C26.1, C27.1, C28.1, C29.1, C30.1, C31.2, C32.1, C33.2, C34.2, IC4.GND, MOD2.GND, R12.2, R16.1, XT2.2, XT2.4; no longer C10.2, C11.1, C12.1, C13.1, C14.1, C15.1, C16.1, C17.1, C18.2, C19.2, C20.1, C7.1, C8.1, C9.1, IC3.GND, MOD1.GND, R10.1, R6.2, XT1.2, XT1.4
- net IO0: now also IC4.GPIO0, MOD2.IO0, R14.2; no longer IC3.GPIO0, MOD1.IO0, R8.2
- net IO12: now also IC4.MTDI, MOD2.IO12; no longer IC3.MTDI, MOD1.IO12
- net IO13: now also IC4.MTCK, MOD2.IO13; no longer IC3.MTCK, MOD1.IO13
- net IO14: now also IC4.MTMS, MOD2.IO14; no longer IC3.MTMS, MOD1.IO14
- net IO15: now also IC4.MTDO, MOD2.IO15, R16.2; no longer IC3.MTDO, MOD1.IO15, R10.2
- net IO1_TX: now also IC4.U0TXD, MOD2.TXD/IO1; no longer IC3.U0TXD, MOD1.TXD/IO1
- net IO2: now also IC4.GPIO2, MOD2.IO2, R15.2; no longer IC3.GPIO2, MOD1.IO2, R9.2
- net IO3_RX: now also IC4.U0RXD, MOD2.RXD/IO3; no longer IC3.U0RXD, MOD1.RXD/IO3
- net IO4: now also IC4.GPIO4, MOD2.IO4; no longer IC3.GPIO4, MOD1.IO4
- net IO5: now also IC4.GPIO5, MOD2.IO5; no longer IC3.GPIO5, MOD1.IO5
- net RST_C: now also C30.2, IC4.EXT_RSTB, R17.1; no longer C20.2, IC3.EXT_RSTB, R11.1
- net RST_M: now also MOD2.RST; no longer MOD1.RST
- net VCC: now also C25.2, C26.2, C27.2, C28.2, C29.2, C31.1, C32.2, C33.1, C34.1, IC4.VDD3P3_1, IC4.VDD3P3_2, IC4.VDDA_1, IC4.VDDA_2, IC4.VDDD, IC4.VDDPST_1, IC4.VDDPST_2, MOD2.VCC, R13.1, R14.1, R15.1, R17.2; no longer C10.1, C12.2, C13.2, C14.2, C15.2, C16.2, C17.2, C18.1, C19.1, IC3.VDD3P3_1, IC3.VDD3P3_2, IC3.VDDA_1, IC3.VDDA_2, IC3.VDDD, IC3.VDDPST_1, IC3.VDDPST_2, MOD1.VCC, R11.2, R7.1, R8.1, R9.1
- net XTAL_IN: now also C23.2, IC4.XTAL_IN, XT2.1; no longer C7.2, IC3.XTAL_IN, XT1.1
- net XTAL_OUT: now also C24.2, IC4.XTAL_OUT, XT2.3; no longer C11.2, IC3.XTAL_OUT, XT1.3
