File: projects/electroniccats_solderingchallenge/version_current/working/working.kicad_pcb (KiCad board)
At the start: 2 copper layers, 33.5 x 33.5 mm, 28 parts, among them J1 ISP, U1 ATtiny85-20SU

Commit message: resyncing
Other:
- net class Default added: clearance 0.2, trace_width 0.35, via_dia 1, via_drill 0.6
- net class vcc added: clearance 0.3, trace_width 0.5, via_dia 1, via_drill 0.6

Commit message: comitting after 1 generations
Other:
- net class Default removed
- net class vcc removed
